Commit message: Changed file-path. Deactivated gazebo-gui. Added comments for simulation

File: universal_robot/ur_description/urdf/common.gazebo.xacro (robot description, xacro)
@@ -3,4 +3,5 @@
   <gazebo>
     <plugin name="ros_control" filename="libgazebo_ros_control.so">
+      <legacyModeNS>true</legacyModeNS>
       <!--robotNamespace>/</robotNamespace-->
       <!--robotSimType>gazebo_ros_control/DefaultRobotHWSim</robotSimType-->

File: universal_robot/ur_description/urdf/eef.urdf (robot description, URDF)
Before this commit: robot eef, 3 links, 0 joints
Links:
- link eef: geometry collision mesh filename=package://ur_description/meshes/EEF.STL scale=0.001 0.001 0.001; visual mesh filename=package://ur_description/meshes/EEF.STL scale=0.001 0.001 0.001

File: universal_robot/ur_description/urdf/ur5_joint_limited_robot.urdf.xacro (robot description, xacro)
@@ -16,5 +16,6 @@
   />
   <!-- Controlbox -->
-  <xacro:include filename="$(find ur_description)/urdf/controlbox.urdf" />
+                                                                                  <!-- COMMENT FOR SIMULATION -->
+  <!--<xacro:include filename="$(find ur_description)/urdf/controlbox.urdf" />-->
   <!-- EEF -->
   <xacro:include filename="$(find ur_description)/urdf/eef.urdf" />
@@ -25,10 +26,11 @@
     <origin xyz="0.0 0.0 0.0" rpy="0.0 0.0 0.0" />
   </joint>
-  <!-- Connection controlbox to MiR -->
-  <joint name="boxJoint" type="fixed">
+  <!-- Connection controlbox to UR -->
+                                                                                  <!-- COMMENT FOR SIMULATION -->
+  <!--<joint name="boxJoint" type="fixed">
     <origin xyz="-0.11 0.038 ${-0.54/2}" rpy="0 0 0" />
     <parent link="base_link" />
     <child link="controlbox" />
-  </joint>
+  </joint>-->
   <!-- Connection UR to EEF -->
   <joint name="eef_fixed_joint" type="fixed">
