Commit message: Changed base_link to base_link_ur

File: universal_robot/ur_description/urdf/ur5.urdf.xacro (robot description, xacro)
@@ -74,5 +74,5 @@
     <xacro:property name="forearm_radius" value="0.040" />    <!-- manually measured -->
     <xacro:property name="wrist_radius" value="0.045" />      <!-- manually measured -->
-    <link name="${prefix}base_link" >
+    <link name="${prefix}base_link_ur" >
       <visual>
         <geometry>
@@ -93,5 +93,5 @@
     </link>
     <joint name="${prefix}shoulder_pan_joint" type="revolute">
-      <parent link="${prefix}base_link" />
+      <parent link="${prefix}base_link_ur" />
       <child link = "${prefix}shoulder_link" />
       <origin xyz="0.0 0.0 ${shoulder_height}" rpy="0.0 0.0 0.0" />
@@ -301,5 +301,5 @@
       -->
       <origin xyz="0 0 0" rpy="0 0 ${-pi}"/>
-      <parent link="${prefix}base_link"/>
+      <parent link="${prefix}base_link_ur"/>
       <child link="${prefix}base"/>
     </joint>

File: universal_robot/ur_description/urdf/ur5_joint_limited_robot.urdf.xacro (robot description, xacro)
@@ -39,5 +39,5 @@
   <joint name="boxJoint" type="fixed">
     <origin xyz="-0.11 0.038 ${-0.54/2}" rpy="0 0 0" />
-    <parent link="base_link" />
+    <parent link="base_link_ur" />
     <child link="controlbox" />
   </joint>

File: universal_robot/ur_description/urdf/ur5_robot.urdf.xacro (robot description, xacro)
@@ -15,5 +15,5 @@
   <joint name="world_joint" type="fixed">
     <parent link="world" />
-    <child link = "base_link" />
+    <child link = "base_link_ur" />
     <origin xyz="0.0 0.0 0.0" rpy="0.0 0.0 0.0" />
   </joint>
@@ -21,5 +21,5 @@
   <joint name="boxJoint" type="fixed">
     <origin xyz="0.038 0 0.352" rpy="0 0 0" />
-    <parent link="base_link" />
+    <parent link="base_link_ur" />
     <child link="controlbox" />
   </joint>
