Commit message: Changes for real robot

File: universal_robot/ur_description/urdf/ur5_joint_limited_robot.urdf.xacro (robot description, xacro)
@@ -17,5 +17,5 @@
   <!-- Controlbox -->
                                                                                   <!-- COMMENT FOR SIMULATION -->
-  <!--<xacro:include filename="$(find ur_description)/urdf/controlbox.urdf" />-->
+  <xacro:include filename="$(find ur_description)/urdf/controlbox.urdf" />
   <!-- EEF -->
   <xacro:include filename="$(find ur_description)/urdf/eef.urdf" />
@@ -28,9 +28,9 @@
   <!-- Connection controlbox to UR -->
                                                                                   <!-- COMMENT FOR SIMULATION -->
-  <!--<joint name="boxJoint" type="fixed">
+  <joint name="boxJoint" type="fixed">
     <origin xyz="-0.11 0.038 ${-0.54/2}" rpy="0 0 0" />
     <parent link="base_link" />
     <child link="controlbox" />
-  </joint>-->
+  </joint>
   <!-- Connection UR to EEF -->
   <joint name="eef_fixed_joint" type="fixed">

Commit message: minor change

File: universal_robot/ur_description/urdf/ur5_joint_limited_robot.urdf.xacro (robot description, xacro)
@@ -32,5 +32,5 @@
   <joint name="world_joint" type="fixed">
     <parent link="world" />
-    <child link = "base_link" />
+    <child link = "base_link_ur" />
     <origin xyz="0.0 0.0 0.0" rpy="0.0 0.0 0.0" />
   </joint>
